Commit message: modifiing lidar config

File: src/solver_description/urdf/lidar.xacro (robot description, xacro)
@@ -35,5 +35,5 @@
         <scan>
           <horizontal>
-            <samples>720</samples>
+            <samples>360</samples>
             <resolution>1</resolution>
             <min_angle>-3.14</min_angle>
@@ -43,5 +43,5 @@
         <range>
           <min>0.4</min>
-          <max>10</max>
+          <max>12</max>
           <resolution>0.01</resolution>
         </range>

File: src/solver_description/urdf/solver_body.xacro (robot description, xacro)
@@ -24,5 +24,4 @@
   <xacro:property name="I_wheel" value="-${(1.0/12.0) * wheel_mass * (3.0 * wheel_link_radius_sq + wheel_link_length * wheel_link_length)}"/>
   <!-- This macro defines the complete inertial section of the wheel -->
-  <!-- it's used later in the code -->
   <xacro:macro name="inertia_wheel">
       <inertial>

File: src/solver_description/urdf/solver_wheel.xacro (robot description, xacro)
@@ -1,9 +1,14 @@
 <?xml version="1.0"?>
 <robot xmlns:xacro="http://ros.org/wiki/xacro" name="solver_wheel">
-	<xacro:macro name="solver_wheel" params="wheel_prefix link_visual_origin_r:=1.570795 joint_origin_x:=${-body_link_x_dim/2+1.2*wheel_link_radius -0.05} joint_origin_y:=${-body_link_y_dim/2 -wheel_link_length/2 } joint_origin_yaw:=${pi_const/2} joint_axis:=1">
+	<xacro:macro name="solver_wheel" params="wheel_prefix link_visual_origin_r:=1.570795
+	joint_origin_x:=${-body_link_x_dim/2+1.2*wheel_link_radius -0.05}
+	joint_origin_y:=${-body_link_y_dim/2 -wheel_link_length/2 }
+	joint_origin_yaw:=${pi_const/2}
+	joint_axis:=1">
 		<joint name="wheel${wheel_prefix}_joint" type="continuous" >
 			<parent link="body_link"/>
 			<child  link="wheel${wheel_prefix}_link" />
-			<origin xyz="${joint_origin_x} ${joint_origin_y} ${wheel_link_z_location }" rpy="0 0 ${joint_origin_yaw}" />
+			<origin xyz="${joint_origin_x} ${joint_origin_y} ${wheel_link_z_location }"
+			rpy="0 0 ${joint_origin_yaw}" />
 			<axis xyz="${joint_axis} 0 0"/>
 			<limit effort="1000" velocity="1000"/>
